Commit message: Update arm mounting point with measurements from AL

File: motive_description/urdf/msa6_v03_on_stand.urdf.xacro (robot description, xacro)
@@ -8,5 +8,5 @@
     <parent link="world" />
     <child link = "base_link" />
-    <origin xyz="0.06985 0.0 1.58115" rpy="1.5708 0 1.5708" />
+    <origin xyz="0.194 0.369 1.73" rpy="1.5708 0 1.5708" />
   </joint>
   <link name="world" />

Commit message: Adjust tcp translation

File: motive_description/urdf/msa6_v03_on_stand.urdf.xacro (robot description, xacro)
@@ -27,5 +27,5 @@
     <parent link="link_L6" />
     <child link = "tcp" />
-    <origin xyz="0 0 0.2" rpy="0 ${-pi/2} 0" />
+    <origin xyz="0 0 0.34" rpy="0 ${-pi/2} 0" />
   </joint>
   <link name="tcp" />
